File: esp32-cam-emmc.kicad_sch (KiCad schematic)
At the start: 47 parts, among them J301 FH34SRJ-24S-0.5SH50, Q107 IRF7606TRPBF, SW102 3.5x2.6 Tact SW, SW103 3.5x2.6 Tact SW, U104 ESP32-S3-WROOM-1-N16R8, U302 MCP1700T-1502E/TT, U303 MCP1700T-2802E/TT, U604 FEMC064G-M11, Y101 32.7680KHz

Commit message: Change Regulator IC and Pullup R
Parts:
- R102: value 10K -> 100K
Changed lines of the file:
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@@
 			)
 		)
-		(property "Value" "10K"
+		(property "Value" "100K"
 			(at 191.77 157.48 0)
 			(effects
@@
 			)
 		)
-		(property "Value" "10K"
+		(property "Value" "100K"
 			(at 171.45 119.38 0)
 			(effects
@@
 			)
 		)
-		(property "Value" "10K"
+		(property "Value" "100K"
 			(at 160.02 157.48 0)
 			(effects
@@
 			)
 		)
-		(property "Value" "10K"
+		(property "Value" "100K"
 			(at 187.96 119.38 0)
 			(effects
@@
 			)
 		)
-		(property "Value" "10K"
+		(property "Value" "100K"
 			(at 167.64 157.48 0)
 			(effects
@@
 			)
 		)
-		(property "Value" "10K"
+		(property "Value" "100K"
 			(at 182.88 157.48 0)
 			(effects
@@
 			)
 		)
-		(property "Value" "10K"
+		(property "Value" "100K"
 			(at 163.83 119.38 0)
 			(effects
@@
 			)
 		)
-		(property "Value" "10K"
+		(property "Value" "100K"
 			(at 175.26 157.48 0)
 			(effects
@@
 			)
 		)
-		(property "Value" "10K"
+		(property "Value" "100K"
 			(at 179.07 119.38 0)
 			(effects
@@
 			)
 		)
-		(property "Value" "10K"
+		(property "Value" "100K"
 			(at 156.21 119.38 0)
 			(effects
